Commit message: mimic joint test

File: My_asset/Crank_slider_system_description/urdf/Crank_slider_system_macro.urdf.xacro (robot description, xacro)
@@ -5,6 +5,6 @@
 <xacro:include filename="../urdf/Crank_slider_system.trans" />
 <xacro:include filename="../urdf/Crank_slider_system.gazebo" />
-<link name="base_link"/>
-<link name="braket1">
+<link name="${prefix}base_link"/>
+<link name="${prefix}braket1">
   <inertial>
     <origin xyz="0.0 0.004999999999999999 0.0" rpy="0 0 0"/>
@@ -26,5 +26,5 @@
   </collision>
 </link>
-<link name="braket2">
+<link name="${prefix}braket2">
   <inertial>
     <origin xyz="5.958400717265278e-10 0.030000000000000002 0.0" rpy="0 0 0"/>
@@ -46,5 +46,5 @@
   </collision>
 </link>
-<link name="motor">
+<link name="${prefix}motor">
   <inertial>
     <origin xyz="5.960465176979568e-10 -5.227138166752354e-13 0.012249999999999872" rpy="0 0 0"/>
@@ -66,5 +66,5 @@
   </collision>
 </link>
-<link name="motor_link">
+<link name="${prefix}motor_link">
   <inertial>
     <origin xyz="5.960465176979568e-10 -5.227138166752354e-13 0.00974999999999987" rpy="0 0 0"/>
@@ -86,5 +86,5 @@
   </collision>
 </link>
-<link name="Link1">
+<link name="${prefix}Link1">
   <inertial>
     <origin xyz="0.01000000059602428 1.249000902703301e-16 -0.005000000000000143" rpy="0 0 0"/>
@@ -106,5 +106,5 @@
   </collision>
 </link>
-<link name="Link2">
+<link name="${prefix}Link2">
   <inertial>
     <origin xyz="0.04700000059604126 2.8449465006019636e-16 0.004999999999999838" rpy="0 0 0"/>
@@ -126,5 +126,5 @@
   </collision>
 </link>
-<link name="Link3">
+<link name="${prefix}Link3">
   <inertial>
     <origin xyz="0.01118519260242784 1.3877787807814457e-16 -0.004999999999988708" rpy="0 0 0"/>
@@ -146,5 +146,5 @@
   </collision>
 </link>
-<link name="Shaft">
+<link name="${prefix}Shaft">
   <inertial>
     <origin xyz="0.04565824322633355 1.0408340855860843e-16 -1.687538997430238e-14" rpy="0 0 0"/>
@@ -166,5 +166,5 @@
   </collision>
 </link>
-<link name="Impact_Plate">
+<link name="${prefix}Impact_Plate">
   <inertial>
     <origin xyz="0.005009856778224464 1.3808398868775384e-15 -5.551115123125783e-17" rpy="0 0 0"/>
@@ -186,5 +186,5 @@
   </collision>
 </link>
-<link name="Slider_jig">
+<link name="${prefix}Slider_jig">
   <inertial>
     <origin xyz="5.96050764301026e-10 0.014032687941284544 -8.326672684688674e-17" rpy="0 0 0"/>
@@ -206,5 +206,5 @@
   </collision>
 </link>
-<link name="Wall">
+<link name="${prefix}Wall">
   <inertial>
     <origin xyz="-0.013718626738737638 0.02626691996491727 1.942890293094024e-16" rpy="0 0 0"/>
@@ -226,5 +226,5 @@
   </collision>
 </link>
-<link name="Slider_jig">
+<link name="${prefix}Slider_jig">
   <inertial>
     <origin xyz="0.014000000596050721 -0.018967312058715453 -0.012000000000000066" rpy="0 0 0"/>
@@ -246,5 +246,5 @@
   </collision>
 </link>
-<link name="Slider1">
+<link name="${prefix}Slider1">
   <inertial>
     <origin xyz="0.021500000596053115 0.0021856845849656595 0.0011086680128989113" rpy="0 0 0"/>
@@ -266,71 +266,71 @@
   </collision>
 </link>
-<joint name="Rigid 44" type="fixed">
+<joint name="${prefix}Rigid 44" type="fixed">
   <origin xyz="0.11 0.01 -0.185" rpy="0 0 0"/>
-  <parent link="base_link"/>
-  <child link="braket1"/>
-</joint>
-<joint name="Rigid 45" type="fixed">
+  <parent link="${prefix}base_link"/>
+  <child link="${prefix}braket1"/>
+</joint>
+<joint name="${prefix}Rigid 45" type="fixed">
   <origin xyz="0.0 0.01 0.025" rpy="0 0 0"/>
-  <parent link="braket1"/>
-  <child link="braket2"/>
-</joint>
-<joint name="Rigid 46" type="fixed">
+  <parent link="${prefix}braket1"/>
+  <child link="${prefix}braket2"/>
+</joint>
+<joint name="${prefix}Rigid 46" type="fixed">
   <origin xyz="0.0 0.03 -0.003" rpy="0 0 0"/>
-  <parent link="braket2"/>
-  <child link="motor"/>
-</joint>
-<joint name="Revolute 47" type="continuous">
+  <parent link="${prefix}braket2"/>
+  <child link="${prefix}motor"/>
+</joint>
+<joint name="${prefix}Revolute 47" type="continuous">
   <origin xyz="0.0 0.0 0.0" rpy="0 0 0"/>
-  <parent link="motor"/>
-  <child link="motor_link"/>
+  <parent link="${prefix}motor"/>
+  <child link="${prefix}motor_link"/>
   <axis xyz="0.0 0.0 1.0"/>
 </joint>
-<joint name="Rigid 48" type="fixed">
+<joint name="${prefix}Rigid 48" type="fixed">
   <origin xyz="0.0 0.0 0.0195" rpy="0 0 0"/>
-  <parent link="motor"/>
-  <child link="Link1"/>
-</joint>
-<joint name="Revolute 49" type="continuous">
+  <parent link="${prefix}motor"/>
+  <child link="${prefix}Link1"/>
+</joint>
+<joint name="${prefix}Revolute 49" type="continuous">
   <origin xyz="0.02 0.0 0.0" rpy="0 0 0"/>
-  <parent link="Link1"/>
-  <child link="Link2"/>
+  <parent link="${prefix}Link1"/>
+  <child link="${prefix}Link2"/>
   <axis xyz="-0.0 -0.0 -1.0"/>
 </joint>
-<joint name="Revolute 50" type="continuous">
+<joint name="${prefix}Revolute 50" type="continuous">
   <origin xyz="0.094 0.0 0.0" rpy="0 0 0"/>
-  <parent link="Link2"/>
-  <child link="Link3"/>
+  <parent link="${prefix}Link2"/>
+  <child link="${prefix}Link3"/>
   <axis xyz="0.0 -0.0 -1.0"/>
 </joint>
-<joint name="Rigid 51" type="fixed">
+<joint name="${prefix}Rigid 51" type="fixed">
   <origin xyz="0.027 0.0 -0.005" rpy="0 0 0"/>
-  <parent link="Link3"/>
-  <child link="Shaft"/>
-</joint>
-<joint name="Rigid 53" type="fixed">
+  <parent link="${prefix}Link3"/>
+  <child link="${prefix}Shaft"/>
+</joint>
+<joint name="${prefix}Rigid 53" type="fixed">
   <origin xyz="0.1 0.0 0.0" rpy="0 0 0"/>
-  <parent link="Shaft"/>
-  <child link="Impact_Plate"/>
-</joint>
-<joint name="Rigid 54" type="fixed">
+  <parent link="${prefix}Shaft"/>
+  <child link="${prefix}Impact_Plate"/>
+</joint>
+<joint name="${prefix}Rigid 54" type="fixed">
   <origin xyz="0.269 0.043 -0.1355" rpy="0 0 0"/>
-  <parent link="base_link"/>
-  <child link="Slider_jig"/>
-</joint>
-<joint name="Rigid 55" type="fixed">
+  <parent link="${prefix}base_link"/>
+  <child link="${prefix}Slider_jig"/>
+</joint>
+<joint name="${prefix}Rigid 55" type="fixed">
   <origin xyz="0.394243 0.01 -0.16" rpy="0 0 0"/>
-  <parent link="base_link"/>
-  <child link="Wall"/>
-</joint>
-<joint name="Rigid 59" type="fixed">
+  <parent link="${prefix}base_link"/>
+  <child link="${prefix}Wall"/>
+</joint>
+<joint name="${prefix}Rigid 59" type="fixed">
   <origin xyz="0.0075 -0.007 0.013" rpy="0 0 0"/>
-  <parent link="Slider1"/>
-  <child link="Slider_jig"/>
-</joint>
-<joint name="Slider 60" type="prismatic">
+  <parent link="${prefix}Slider1"/>
+  <child link="${prefix}Slider_jig"/>
+</joint>
+<joint name="${prefix}Slider 60" type="prismatic">
   <origin xyz="0.0105 0.0 0.0" rpy="0 0 0"/>
-  <parent link="Shaft"/>
-  <child link="Slider1"/>
+  <parent link="${prefix}Shaft"/>
+  <child link="${prefix}Slider1"/>
   <axis xyz="-1.0 -0.0 -0.0"/>
   <limit upper="0.0" lower="0.0" effort="100" velocity="100"/>

File: My_asset/Crank_slider_system_description1/urdf/Crank_slider_system.xacro (robot description, xacro)
@@ -1,7 +1,7 @@
 <?xml version="1.0" ?>
 <robot name="Crank_slider_system" xmlns:xacro="http://www.ros.org/wiki/xacro">
-<xacro:include filename="$(find Crank_slider_system_description)/urdf/materials.xacro" />
-<xacro:include filename="$(find Crank_slider_system_description)/urdf/Crank_slider_system.trans" />
-<xacro:include filename="$(find Crank_slider_system_description)/urdf/Crank_slider_system.gazebo" />
+<xacro:include filename="../urdf/materials.xacro" />
+<xacro:include filename="../urdf/Crank_slider_system.trans" />
+<xacro:include filename="../urdf/Crank_slider_system.gazebo" />
 <link name="base_link">
   <inertial>
