Commit message: Crank slider system copy - joint type change

File: My_asset/Crank_slider_system_description/urdf/Crank_slider_system.urdf (robot description, URDF)
Before this commit: robot Crank_slider_system, 13 links, 12 joints
Links:
- link Impact_Plate: geometry collision mesh filename=../col_meshes/Impact_Plate.stl scale=0.001 0.001 0.001; visual mesh filename=../vis_mesh/Impact_Plate.stl scale=0.001 0.001 0.001
- link Link1: geometry collision mesh filename=../col_meshes/Link1.stl scale=0.001 0.001 0.001; visual mesh filename=../vis_mesh/Link1.stl scale=0.001 0.001 0.001
- link Link2: geometry collision mesh filename=../col_meshes/Link2.stl scale=0.001 0.001 0.001; visual mesh filename=../vis_mesh/Link2.stl scale=0.001 0.001 0.001
- link Link3: geometry collision mesh filename=../col_meshes/Link3.stl scale=0.001 0.001 0.001; visual mesh filename=../vis_mesh/Link3.stl scale=0.001 0.001 0.001
- link Shaft: geometry collision mesh filename=../col_meshes/Shaft.stl scale=0.001 0.001 0.001; visual mesh filename=../vis_mesh/Shaft.stl scale=0.001 0.001 0.001
- link Slider1: geometry collision mesh filename=../col_meshes/Slider1.stl scale=0.001 0.001 0.001; visual mesh filename=../vis_mesh/Slider1.stl scale=0.001 0.001 0.001
- link Slider_jig: geometry collision mesh filename=../col_meshes/Slider_jig.stl scale=0.001 0.001 0.001; visual mesh filename=../vis_mesh/Slider_jig.stl scale=0.001 0.001 0.001
- link Wall: geometry collision mesh filename=../col_meshes/Wall.stl scale=0.001 0.001 0.001; visual mesh filename=../vis_mesh/Wall.stl scale=0.001 0.001 0.001
- link base_link: geometry collision mesh filename=../col_meshes/base_link.stl scale=0.001 0.001 0.001; visual mesh filename=../vis_mesh/base_link.stl scale=0.001 0.001 0.001
- link braket1: geometry collision mesh filename=../col_meshes/braket1.stl scale=0.001 0.001 0.001; visual mesh filename=../vis_mesh/braket1.stl scale=0.001 0.001 0.001
- link braket2: geometry collision mesh filename=../col_meshes/braket2.stl scale=0.001 0.001 0.001; visual mesh filename=../vis_mesh/braket2.stl scale=0.001 0.001 0.001
- link motor: geometry collision mesh filename=../col_meshes/motor.stl scale=0.001 0.001 0.001; visual mesh filename=../vis_mesh/motor.stl scale=0.001 0.001 0.001
- link motor_shaft: geometry collision mesh filename=../col_meshes/motor_shaft.stl scale=0.001 0.001 0.001; visual mesh filename=../vis_mesh/motor_shaft.stl scale=0.001 0.001 0.001
Joints:
- removed joint Slider 60
- added joint Rigid 54: type fixed, parent base_link, child Slider_jig, origin xyz=0.269 0.043 -0.1355 rpy=0 0 0
- joint Rigid 59: child Slider_jig -> Slider1; parent Slider1 -> Slider_jig

File: My_asset/TEST_LINK_sizeup_description/urdf/TEST_LINK_sizeup.xacro (robot description, xacro)
@@ -1,7 +1,7 @@
 <?xml version="1.0" ?>
 <robot name="TEST_LINK_sizeup" xmlns:xacro="http://www.ros.org/wiki/xacro">
-<xacro:include filename="$(find TEST_LINK_sizeup_description)/urdf/materials.xacro" />
-<xacro:include filename="$(find TEST_LINK_sizeup_description)/urdf/TEST_LINK_sizeup.trans" />
-<xacro:include filename="$(find TEST_LINK_sizeup_description)/urdf/TEST_LINK_sizeup.gazebo" />
+<xacro:include filename="../urdf/materials.xacro" />
+<xacro:include filename="../urdf/TEST_LINK_sizeup.trans" />
+<xacro:include filename="../urdf/TEST_LINK_sizeup.gazebo" />
 <link name="base_link">
   <inertial>
@@ -13,5 +13,6 @@
     <origin xyz="0 0 0" rpy="0 0 0"/>
     <geometry>
-      <mesh filename="package://TEST_LINK_sizeup_description/meshes/base_link.stl" scale="0.001 0.001 0.001"/>
+      <!--0.001 means, mm -> m-->
+      <mesh filename="../meshes/base_link.stl" scale="0.001 0.001 0.001"/>
     </geometry>
     <material name="silver"/>
@@ -20,5 +21,5 @@
     <origin xyz="0 0 0" rpy="0 0 0"/>
     <geometry>
-      <mesh filename="package://TEST_LINK_sizeup_description/meshes/base_link.stl" scale="0.001 0.001 0.001"/>
+      <mesh filename="../meshes/base_link.stl" scale="0.001 0.001 0.001"/>
     </geometry>
   </collision>

File: My_asset/TEST_LINK_sizeup_description/urdf/materials.xacro (robot description, xacro)
@@ -1,6 +1,7 @@
 <?xml version="1.0" ?>
 <robot name="TEST_LINK_sizeup" xmlns:xacro="http://www.ros.org/wiki/xacro" >
-<material name="silver">
-  <color rgba="0.700 0.700 0.700 1.000"/>
+<material name="black">
+  <color rgba="0.000 0.000 0.000 1.000"/>
+  <!--<color rgba="0.700 0.700 0.700 1.000"/>-->
 </material>
 </robot>

Commit message: 20250903

File: My_asset/Crank_slider_system_description/urdf/Crank_slider_system.urdf (robot description, URDF)
Before this commit: robot Crank_slider_system, 13 links, 12 joints
Joints:
- added joint Slider 60: type prismatic, parent Shaft, child Slider1, origin xyz=0.0105 0.0 0.0 rpy=0 0 0, axis -1.0 -0.0 -0.0, mimic joint=Revolute 49
