Commit message: video add

File: My_asset/Crank_slider_system_copy_description/urdf/Crank_slider_system_copy.urdf (robot description, URDF)
Before this commit: robot Crank_slider_system_copy, 13 links, 12 joints
Joints:
- removed joint Rigid 44
- added joint Rigid44: type fixed, parent base_link, child braket1_1, origin xyz=0.11 0.01 -0.185 rpy=0 0 0

Commit message: 20250827

File: My_asset/Crank_slider_system_copy_description/urdf/Crank_slider_system_copy.urdf (robot description, URDF)
Before this commit: robot Crank_slider_system_copy, 13 links, 12 joints
Joints:
- added joint Slider 60: type prismatic, parent Shaft_1, child Slider1_1, origin xyz=0.0105 0.0 0.0 rpy=0 0 0, axis -1.0 -0.0 -0.0, limit lower=0.0 upper=0.0 effort=100 velocity=100, mimic joint=Revolute 47 multiplier=-0.5 offset=0.0

Commit message: 2025.09.01 backup

File: My_asset/Crank_slider_system_copy_description/urdf/Crank_slider_system_copy.urdf (robot description, URDF)
Before this commit: robot Crank_slider_system_copy, 13 links, 13 joints
Links:
- link Slider_jig_1: mass 0.29233817695735465 -> 2000000
Joints:
- removed joint Rigid 61

File: My_asset/Crank_slider_system_description/urdf/Crank_slider_system_copy.urdf (robot description, URDF)
Before this commit: robot Crank_slider_system, 13 links, 12 joints
Links:
- link Slider_jig: mass 0.29233817695735465 -> 2000
